File: Hardware/Spectacle_Audio_Output_Board.brd (EAGLE design)
At the start: 25.4 x 55.9 mm, 86 parts, among them J4 AUDIO-JACK3, J5 AUDIO-JACK3, U1 CY8C4146LQI-S422, U2 3.3V, U3 3.3V, U4 AT25SF041-SOIC8, U5 VS1000, U6 SN74LVC1G66, U7 SN74LVC1G66, Y1 12MHz

Commit message: Touch ups before v10 double check
Parts:
- J3: value (none) -> AUDIO_JACK_3.5MM_SMD
- J4, J5: value AUDIO-JACK3 -> AUDIO_JACK_TRRSSMD_RA; device SparkFun-Connectors:AUDIO-JACK-TRRS-SMD -> SparkFun-Connectors:AUDIO_JACK_3.5MM_TRRS_SMD_RA
Changed lines of the file:
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@@
 <grid distance="0.05" unitdist="inch" unit="inch" style="lines" multiple="1" display="yes" altdistance="0.005" altunitdist="inch" altunit="inch"/>
 <layers>
-<layer number="1" name="Top" color="4" fill="1" visible="yes" active="yes"/>
+<layer number="1" name="Top" color="4" fill="1" visible="no" active="yes"/>
 <layer number="2" name="Route2" color="1" fill="3" visible="no" active="yes"/>
 <layer number="15" name="Route15" color="4" fill="6" visible="no" active="yes"/>
@@
 <layer number="19" name="Unrouted" color="6" fill="1" visible="yes" active="yes"/>
 <layer number="20" name="Dimension" color="15" fill="1" visible="yes" active="yes"/>
-<layer number="21" name="tPlace" color="16" fill="1" visible="yes" active="yes"/>
+<layer number="21" name="tPlace" color="16" fill="1" visible="no" active="yes"/>
 <layer number="22" name="bPlace" color="14" fill="1" visible="yes" active="yes"/>
-<layer number="23" name="tOrigins" color="15" fill="1" visible="yes" active="yes"/>
+<layer number="23" name="tOrigins" color="15" fill="1" visible="no" active="yes"/>
 <layer number="24" name="bOrigins" color="15" fill="1" visible="yes" active="yes"/>
 <layer number="25" name="tNames" color="7" fill="1" visible="no" active="yes"/>
@@
 <layer number="43" name="vRestrict" color="2" fill="10" visible="no" active="yes"/>
 <layer number="44" name="Drills" color="7" fill="1" visible="no" active="yes"/>
-<layer number="45" name="Holes" color="7" fill="1" visible="yes" active="yes"/>
+<layer number="45" name="Holes" color="7" fill="1" visible="no" active="yes"/>
 <layer number="46" name="Milling" color="3" fill="1" visible="no" active="yes"/>
 <layer number="47" name="Measures" color="7" fill="1" visible="no" active="yes"/>
 <layer number="48" name="Document" color="7" fill="1" visible="no" active="yes"/>
 <layer number="49" name="Reference" color="7" fill="1" visible="no" active="yes"/>
-<layer number="51" name="tDocu" color="6" fill="1" visible="yes" active="yes"/>
+<layer number="51" name="tDocu" color="6" fill="1" visible="no" active="yes"/>
 <layer number="52" name="bDocu" color="7" fill="1" visible="no" active="yes"/>
 <layer number="3" name="Route3" color="4" fill="3" visible="no" active="no"/>
@@
 <attribute name="PROD_ID" value="RES-07856" x="19.05" y="30.226" size="1.778" layer="27" font="vector" ratio="15" rot="R180" display="off"/>
 </element>
-<element name="J4" library="SparkFun-Connectors" package="AUDIO-JACK-TRRS-SMD" value="AUDIO-JACK3" x="0" y="20.32">
+<element name="J4" library="SparkFun-Connectors" package="AUDIO_JACK_3.5MM_TRRS_SMD_RA" value="AUDIO_JACK_TRRSSMD_RA" x="0" y="20.32">
 <attribute name="PROD_ID" value="CONN-10676" x="0" y="20.32" size="1.778" layer="27" display="off"/>
+<attribute name="SF_ID" value="PRT-12639" x="0" y="20.32" size="1.778" layer="27" display="off"/>
 </element>
 <element name="D4" library="SparkFun-DiscreteSemi" package="SOT23-3" value="PESD1CAN" x="5.969" y="27.051">
@@
 <attribute name="PROD_ID" value="CAP-11015" x="6.35" y="16.51" size="1.778" layer="28" font="vector" ratio="15" rot="MR0" display="off"/>
 </element>
-<element name="J5" library="SparkFun-Connectors" package="AUDIO-JACK-TRRS-SMD" value="AUDIO-JACK3" x="0" y="10.16">
+<element name="J5" library="SparkFun-Connectors" package="AUDIO_JACK_3.5MM_TRRS_SMD_RA" value="AUDIO_JACK_TRRSSMD_RA" x="0" y="10.16">
 <attribute name="PROD_ID" value="CONN-10676" x="0" y="10.16" size="1.778" layer="27" display="off"/>
+<attribute name="SF_ID" value="PRT-12639" x="0" y="10.16" size="1.778" layer="27" display="off"/>
 </element>
 <element name="J1" library="SparkFun-Connectors" package="1X06_NO_SILK" value="" x="1.27" y="26.67" rot="R90"/>
@@
 <attribute name="PROD_ID" value="RES-07868" x="18.415" y="15.24" size="1.778" layer="28" font="vector" ratio="15" rot="MR90" display="off"/>
 </element>
-<element name="J3" library="SparkFun-Connectors" package="AUDIO-JACK-3.5MM-SMD" value="" x="0" y="45.72">
+<element name="J3" library="SparkFun-Connectors" package="AUDIO-JACK-3.5MM-SMD" value="AUDIO_JACK_3.5MM_SMD" x="0" y="45.72">
 <attribute name="PROD_ID" value="CONN-10353" x="0" y="45.72" size="1.778" layer="27" font="vector" ratio="15" display="off"/>
 </element>
@@
 <contactref element="R26" pad="2"/>
 <contactref element="R2" pad="2"/>
-<contactref element="J3" pad="SLEEVE"/>
 <via x="21.336" y="49.784" extent="1-16" drill="0.254"/>
 <via x="19.939" y="51.054" extent="1-16" drill="0.254"/>
@@
 <via x="15.113" y="3.048" extent="1-16" drill="0.254"/>
 <via x="12.7" y="8.509" extent="1-16" drill="0.254"/>
+<contactref element="J3" pad="SLEEVE"/>
 </signal>
 <signal name="VCC">
@@
 <contactref element="C13" pad="2"/>
 <contactref element="R20" pad="2"/>
-<contactref element="J3" pad="TIP"/>
 <wire x1="18.327" y1="48.26" x2="18.327" y2="49.784" width="0.2032" layer="1"/>
 <wire x1="18.327" y1="48.26" x2="13.208" y2="48.26" width="0.2032" layer="1"/>
@@
 <wire x1="11.938" y1="44.45" x2="11.684" y2="44.196" width="0.2032" layer="1"/>
 <wire x1="11.684" y1="44.196" x2="11.684" y2="42.286" width="0.2032" layer="1"/>
+<contactref element="J3" pad="TIP"/>
 <wire x1="11.684" y1="42.286" x2="11.7" y2="42.27" width="0.2032" layer="1"/>
 </signal>
@@
 <contactref element="C14" pad="2"/>
 <contactref element="R19" pad="2"/>
-<contactref element="J3" pad="RING"/>
 <wire x1="16.041" y1="41.91" x2="16.041" y2="40.386" width="0.254" layer="1"/>
 <wire x1="16.041" y1="41.91" x2="15.24" y2="41.91" width="0.2032" layer="1"/>
@@
 <wire x1="4.445" y1="50.8" x2="4.318" y2="50.673" width="0.2032" layer="1"/>
 <wire x1="4.318" y1="50.673" x2="4.318" y2="49.188" width="0.2032" layer="1"/>
+<contactref element="J3" pad="RING"/>
 <wire x1="4.318" y1="49.188" x2="4.3" y2="49.17" width="0.2032" layer="1"/>
 </signal>
