File: Production/13506-Spectacle_Audio_Output_Board-panel.10.brd (EAGLE design)
At the start: 185.4 x 126 mm, 999 parts, among them J12 AUDIO_JACK_3.5MM_SMD, J14 AUDIO_JACK_TRRSSMD_RA, J15 AUDIO_JACK_TRRSSMD_RA, J18 AUDIO_JACK_3.5MM_SMD, J20 AUDIO_JACK_TRRSSMD_RA, J21 AUDIO_JACK_TRRSSMD_RA, J24 AUDIO_JACK_3.5MM_SMD, J26 AUDIO_JACK_TRRSSMD_RA, J27 AUDIO_JACK_TRRSSMD_RA, J3 AUDIO_JACK_3.5MM_SMD, J30 AUDIO_JACK_3.5MM_SMD, J32 AUDIO_JACK_TRRSSMD_RA, J33 AUDIO_JACK_TRRSSMD_RA, J36 AUDIO_JACK_3.5MM_SMD, J38 AUDIO_JACK_TRRSSMD_RA, J39 AUDIO_JACK_TRRSSMD_RA, J4 AUDIO_JACK_TRRSSMD_RA, J42 AUDIO_JACK_3.5MM_SMD, J44 AUDIO_JACK_TRRSSMD_RA, J45 AUDIO_JACK_TRRSSMD_RA, J48 AUDIO_JACK_3.5MM_SMD, J5 AUDIO_JACK_TRRSSMD_RA, J50 AUDIO_JACK_TRRSSMD_RA, J51 AUDIO_JACK_TRRSSMD_RA, J54 AUDIO_JACK_3.5MM_SMD, J56 AUDIO_JACK_TRRSSMD_RA, J57 AUDIO_JACK_TRRSSMD_RA, J60 AUDIO_JACK_3.5MM_SMD, J62 AUDIO_JACK_TRRSSMD_RA, J63 AUDIO_JACK_TRRSSMD_RA, J66 AUDIO_JACK_3.5MM_SMD, J68 AUDIO_JACK_TRRSSMD_RA, J69 AUDIO_JACK_TRRSSMD_RA, J72 AUDIO_JACK_3.5MM_SMD, J8 AUDIO_JACK_TRRSSMD_RA, J9 AUDIO_JACK_TRRSSMD_RA, U1 CY8C4146LQI-S422, U10 VS1000, U11 3.3V, U12 AT25SF041-SOIC8, U13 SN74LVC1G66, U14 SN74LVC1G66, U15 CY8C4146LQI-S422, U16 3.3V, U17 VS1000, U18 3.3V, U19 AT25SF041-SOIC8, U2 3.3V, U20 SN74LVC1G66, U21 SN74LVC1G66, U22 CY8C4146LQI-S422, U23 3.3V, U24 VS1000, U25 3.3V, U26 AT25SF041-SOIC8, U27 SN74LVC1G66, U28 SN74LVC1G66, U29 CY8C4146LQI-S422, U3 3.3V, U30 3.3V, U31 VS1000, U32 3.3V, U33 AT25SF041-SOIC8, U34 SN74LVC1G66, U35 SN74LVC1G66, U36 CY8C4146LQI-S422, U37 3.3V, U38 VS1000, U39 3.3V, U4 AT25SF041-SOIC8, U40 AT25SF041-SOIC8, U41 SN74LVC1G66, U42 SN74LVC1G66, U43 CY8C4146LQI-S422, U44 3.3V, U45 VS1000, U46 3.3V, U47 AT25SF041-SOIC8, U48 SN74LVC1G66, U49 SN74LVC1G66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

Commit message: panel
Parts:
- added E$2: (no value), SparkFun-Retired:FIDUCIAL-1.5X3
- added E$3, E$4: (no value), SparkFun-Aesthetics:FIDUCIAL-1X2
Changed lines of the file:
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@@
 <layers>
 <layer number="1" name="Top" color="4" fill="1" visible="yes" active="yes"/>
-<layer number="2" name="Route2" color="1" fill="3" visible="yes" active="yes"/>
-<layer number="15" name="Route15" color="4" fill="6" visible="yes" active="yes"/>
+<layer number="2" name="Route2" color="1" fill="3" visible="no" active="yes"/>
+<layer number="15" name="Route15" color="4" fill="6" visible="no" active="yes"/>
 <layer number="16" name="Bottom" color="1" fill="1" visible="yes" active="yes"/>
 <layer number="17" name="Pads" color="2" fill="1" visible="yes" active="yes"/>
@@
 <layer number="23" name="tOrigins" color="15" fill="1" visible="yes" active="yes"/>
 <layer number="24" name="bOrigins" color="15" fill="1" visible="yes" active="yes"/>
-<layer number="25" name="tNames" color="7" fill="1" visible="yes" active="yes"/>
-<layer number="26" name="bNames" color="7" fill="1" visible="yes" active="yes"/>
-<layer number="27" name="tValues" color="7" fill="1" visible="yes" active="yes"/>
-<layer number="28" name="bValues" color="7" fill="1" visible="yes" active="yes"/>
-<layer number="29" name="tStop" color="7" fill="3" visible="yes" active="yes"/>
-<layer number="30" name="bStop" color="7" fill="6" visible="yes" active="yes"/>
-<layer number="31" name="tCream" color="7" fill="4" visible="yes" active="yes"/>
-<layer number="32" name="bCream" color="7" fill="5" visible="yes" active="yes"/>
-<layer number="39" name="tKeepout" color="4" fill="11" visible="yes" active="yes"/>
-<layer number="40" name="bKeepout" color="1" fill="11" visible="yes" active="yes"/>
-<layer number="41" name="tRestrict" color="4" fill="10" visible="yes" active="yes"/>
-<layer number="42" name="bRestrict" color="1" fill="10" visible="yes" active="yes"/>
-<layer number="43" name="vRestrict" color="2" fill="10" visible="yes" active="yes"/>
-<layer number="44" name="Drills" color="7" fill="1" visible="yes" active="yes"/>
+<layer number="25" name="tNames" color="7" fill="1" visible="no" active="yes"/>
+<layer number="26" name="bNames" color="7" fill="1" visible="no" active="yes"/>
+<layer number="27" name="tValues" color="7" fill="1" visible="no" active="yes"/>
+<layer number="28" name="bValues" color="7" fill="1" visible="no" active="yes"/>
+<layer number="29" name="tStop" color="7" fill="3" visible="no" active="yes"/>
+<layer number="30" name="bStop" color="7" fill="6" visible="no" active="yes"/>
+<layer number="31" name="tCream" color="7" fill="4" visible="no" active="yes"/>
+<layer number="32" name="bCream" color="7" fill="5" visible="no" active="yes"/>
+<layer number="39" name="tKeepout" color="4" fill="11" visible="no" active="yes"/>
+<layer number="40" name="bKeepout" color="1" fill="11" visible="no" active="yes"/>
+<layer number="41" name="tRestrict" color="4" fill="10" visible="no" active="yes"/>
+<layer number="42" name="bRestrict" color="1" fill="10" visible="no" active="yes"/>
+<layer number="43" name="vRestrict" color="2" fill="10" visible="no" active="yes"/>
+<layer number="44" name="Drills" color="7" fill="1" visible="no" active="yes"/>
 <layer number="45" name="Holes" color="7" fill="1" visible="yes" active="yes"/>
-<layer number="46" name="Milling" color="3" fill="1" visible="yes" active="yes"/>
-<layer number="47" name="Measures" color="7" fill="1" visible="yes" active="yes"/>
-<layer number="48" name="Document" color="7" fill="1" visible="yes" active="yes"/>
-<layer number="49" name="Reference" color="7" fill="1" visible="yes" active="yes"/>
+<layer number="46" name="Milling" color="3" fill="1" visible="no" active="yes"/>
+<layer number="47" name="Measures" color="7" fill="1" visible="no" active="yes"/>
+<layer number="48" name="Document" color="7" fill="1" visible="no" active="yes"/>
+<layer number="49" name="Reference" color="7" fill="1" visible="no" active="yes"/>
 <layer number="51" name="tDocu" color="6" fill="1" visible="yes" active="yes"/>
-<layer number="52" name="bDocu" color="7" fill="1" visible="yes" active="yes"/>
+<layer number="52" name="bDocu" color="7" fill="1" visible="no" active="yes"/>
 <layer number="3" name="Route3" color="4" fill="3" visible="no" active="no"/>
 <layer number="4" name="Route4" color="1" fill="4" visible="no" active="no"/>
@@
 <element name="E$8" library="SparkFun-Aesthetics" package="FIDUCIAL-1X2" value="" x="180.467" y="13.208"/>
 <element name="E$1" library="SparkFun-Retired" package="FIDUCIAL-1.5X3" value="" x="4.064" y="11.684"/>
+<element name="E$2" library="SparkFun-Retired" package="FIDUCIAL-1.5X3" value="" x="4.064" y="11.684" rot="MR90"/>
+<element name="E$3" library="SparkFun-Aesthetics" package="FIDUCIAL-1X2" value="" x="180.467" y="13.208" rot="MR0"/>
+<element name="E$4" library="SparkFun-Aesthetics" package="FIDUCIAL-1X2" value="" x="180.467" y="113.284" rot="MR180"/>
 </elements>
 <signals>
